File: hardware/tag/_autosave-tag.kicad_pcb (KiCad board)
At the start: 2 copper layers, 50 x 52 mm, 103 parts, among them J1 USB_C_Receptacle_USB2.0_16P, J2 BATTERY, J3 UART, J4 I2C, J5 STM SWD, J6 ADC, J7 BLE SWD, J8 SOURCE, SW1 SW_Push, SW2 SW_SPDT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

Commit message: wip(hardware): save tag schematic & pcb layout
Parts:
- moved TP4 19.0 mm to (86.2, 74.0)
- moved J5 0.06 mm to (40.4, 91.5)
Routing:
- net /SPI_MOSI: track 32.6 -> 29.5 mm, vias 1 -> 0
- net /UWB_IQR: track 27.2 -> 26.3 mm
- net /SPI_SCK: track 37.6 -> 36.7 mm
- net /SPI_MISO: track 35.9 -> 35.3 mm
- net GND: vias 88 -> 91
Changed lines of the file:
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@@
 		)
 		(embedded_fonts no)
-		(model "${KICAD9_3DMODEL_DIR}/Connector_JST.3dshapes/JST_PH_B2B-PH-K_1x02_P2.00mm_Vertical.step"
+		(model "${KICAD9_3DMODEL_DIR}/Connector_JST.3dshapes/JST_PH_S2B-PH-K_1x02_P2.00mm_Horizontal.step"
 			(offset
 				(xyz 0 0 0)
@@
 	(footprint "TestPoint:TestPoint_Pad_D2.0mm"
 		(layer "F.Cu")
-		(at 104.15 80.2)
+		(at 86.2 74)
 		(descr "SMD pad as test Point, diameter 2.0mm")
 		(tags "test point SMD pad")
@@
 	(footprint "Other_Footprint:JST_BM04B-SRSS-TB_LF__SN_"
 		(layer "F.Cu")
-		(at 40.5 91.5 90)
+		(at 40.4375 91.5 90)
 		(property "Reference" "J5"
 			(at 0 -2.4875 90)
@@
 	)
 	(segment
-		(start 40.5 93)
-		(end 42.275 93)
-		(width 0.25)
-		(layer "F.Cu")
-		(net 1)
-	)
-	(segment
 		(start 71.2 78.7)
 		(end 71.2 84.981425)
@@
 	)
 	(segment
+		(start 42.2125 93)
+		(end 40.5 93)
+		(width 0.25)
+		(layer "F.Cu")
+		(net 1)
+	)
+	(segment
 		(start 44.8 73.8)
 		(end 45 73.6)
@@
 	)
 	(segment
-		(start 56.95 75.0625)
-		(end 56.942595 75.055095)
+		(start 56.75 71.66)
+		(end 56.95 71.86)
 		(width 0.25)
 		(layer "F.Cu")
@@
 	)
 	(segment
-		(start 56.942595 75.055095)
-		(end 56.942595 74.834095)
+		(start 56.75 60.6)
+		(end 56.75 71.66)
 		(width 0.25)
 		(layer "F.Cu")
@@
 	)
 	(segment
-		(start 56.75 59.5)
-		(end 56.75 71.66)
+		(start 51.05 57.8137)
+		(end 53.9637 57.8137)
 		(width 0.25)
 		(layer "F.Cu")
@@
 	)
 	(segment
-		(start 54.825 67.325)
-		(end 49.275 67.325)
+		(start 56.95 75.0625)
+		(end 56.942595 75.055095)
 		(width 0.25)
 		(layer "F.Cu")
@@
 	)
 	(segment
-		(start 51.05 57.8137)
-		(end 55.0637 57.8137)
+		(start 56.942595 75.055095)
+		(end 56.942595 74.834095)
 		(width 0.25)
 		(layer "F.Cu")
@@
 	)
 	(segment
-		(start 49.275 67.325)
-		(end 46.9625 69.6375)
+		(start 54.825 67.325)
+		(end 49.275 67.325)
 		(width 0.25)
 		(layer "F.Cu")
@@
 	)
 	(segment
-		(start 55.05 67.1)
-		(end 54.825 67.325)
+		(start 49.275 67.325)
+		(end 46.9625 69.6375)
 		(width 0.25)
 		(layer "F.Cu")
@@
 	)
 	(segment
-		(start 56.75 71.66)
-		(end 56.95 71.86)
+		(start 55.05 67.1)
+		(end 54.825 67.325)
 		(width 0.25)
 		(layer "F.Cu")
@@
 	)
 	(segment
-		(start 55.0637 57.8137)
-		(end 56.75 59.5)
+		(start 53.9637 57.8137)
+		(end 56.75 60.6)
 		(width 0.25)
 		(layer "F.Cu")
@@
 	)
 	(segment
-		(start 58.55 56.95)
-		(end 58.55 71.43)
+		(start 53.5637 53.6137)
+		(end 58.55 58.6)
 		(width 0.25)
 		(layer "F.Cu")
@@
 	)
 	(segment
-		(start 58.55 71.43)
-		(end 57.95 72.03)
+		(start 57.95 72.03)
+		(end 57.95 75.0625)
 		(width 0.25)
 		(layer "F.Cu")
@@
 	)
 	(segment
-		(start 55.2137 53.6137)
-		(end 58.55 56.95)
+		(start 51.05 53.6137)
+		(end 53.5637 53.6137)
 		(width 0.25)
 		(layer "F.Cu")
@@
 	)
 	(segment
-		(start 51.05 53.6137)
-		(end 55.2137 53.6137)
+		(start 58.55 71.43)
+		(end 57.95 72.03)
 		(width 0.25)
 		(layer "F.Cu")
@@
 	)
 	(segment
-		(start 57.95 72.03)
-		(end 57.95 75.0625)
+		(start 58.55 58.6)
+		(end 58.55 71.43)
 		(width 0.25)
 		(layer "F.Cu")
@@
 	)
 	(segment
-		(start 55.6137 56.4137)
-		(end 57.7 58.5)
+		(start 57.7 60.05)
+		(end 54.0637 56.4137)
 		(width 0.25)
 		(layer "F.Cu")
@@
 	)
 	(segment
-		(start 51.05 56.4137)
-		(end 55.6 56.4137)
-		(width 0.25)
-		(layer "F.Cu")
-		(net 14)
-	)
-	(segment
-		(start 57.7 58.5)
-		(end 57.7 69)
+		(start 54.0637 56.4137)
+		(end 51.05 56.4137)
 		(width 0.25)
 		(layer "F.Cu")
@@
 	)
 	(segment
-		(start 57.45 71.89)
-		(end 57.45 75.0625)
+		(start 57.7 69)
+		(end 57.7 60.05)
 		(width 0.25)
 		(layer "F.Cu")
@@
 	)
 	(segment
-		(start 55.6 56.4137)
-		(end 55.6137 56.4137)
+		(start 57.45 71.89)
+		(end 57.45 75.0625)
 		(width 0.25)
 		(layer "F.Cu")
@@
 	)
 	(segment
-		(start 57.35 68.65)
-		(end 57.7 69)
+		(start 55.05 68.65)
+		(end 57.35 68.65)
 		(width 0.25)
 		(layer "B.Cu")
@@
 	)
 	(segment
-		(start 55.05 68.65)
-		(end 57.35 68.65)
+		(start 57.35 68.65)
+		(end 57.7 69)
 		(width 0.25)
 		(layer "B.Cu")
@@
 	)
 	(segment
-		(start 54.6125 59.2125)
-		(end 55.9 60.5)
-		(width 0.25)
-		(layer "F.Cu")
-		(net 15)
-	)
-	(segment
 		(start 55.9 68.5)
 		(end 55.9 71.48)
@@
 	)
 	(segment
+		(start 53.5625 59.2125)
+		(end 55.9 61.55)
+		(width 0.25)
+		(layer "F.Cu")
+		(net 15)
+	)
+	(segment
 		(start 55.15 67.95)
 		(end 55.35 67.95)
@@
 	(segment
 		(start 51.05 59.2125)
-		(end 54.6125 59.2125)
+		(end 53.5625 59.2125)
 		(width 0.25)
 		(layer "F.Cu")
@@
 	)
 	(segment
-		(start 55.9 68.5)
-		(end 55.9 60.5)
+		(start 55.9 61.55)
+		(end 55.9 68.5)
 		(width 0.25)
 		(layer "F.Cu")
@@
 		(net 15)
 	)
-	(via
-		(at 55.9 60.5)
-		(size 0.7)
-		(drill 0.3)
-		(layers "F.Cu" "B.Cu")
-		(net 15)
-	)
-	(segment
-		(start 55.9 62.95)
-		(end 55.9 60.5)
-		(width 0.25)
-		(layer "B.Cu")
-		(net 15)
-	)
 	(segment
 		(start 54.77429 73.228886)
@@
 	)
 	(via
+		(at 57.6 58.8)
+		(size 0.5)
+		(drill 0.25)
+		(layers "F.Cu" "B.Cu")
+		(free yes)
+		(net 29)
+	)
+	(via
 		(at 50.33128 97.825872)
 		(size 0.5)
@@
 	)
 	(via
+		(at 53.675003 55.05)
+		(size 0.5)
+		(drill 0.25)
+		(layers "F.Cu" "B.Cu")
+		(free yes)
+		(net 29)
+	)
+	(via
 		(at 50.350922 97.075)
 		(size 0.5)
@@
 	)
 	(via
-		(at 55.25 61.45)
+		(at 53.05 55.05)
+		(size 0.5)
+		(drill 0.25)
+		(layers "F.Cu" "B.Cu")
+		(free yes)
+		(net 29)
+	)
+	(via
+		(at 55.15 61.8)
 		(size 0.5)
 		(drill 0.25)
@@
 	)
 	(segment
-		(start 40.5 91)
-		(end 42.275 91)
-		(width 0.2)
+		(start 42.2125 91)
+		(end 40.5 91)
+		(width 0.25)
 		(layer "F.Cu")
 		(net 30)
@@
 	)
 	(segment
-		(start 52.95 81.9375)
-		(end 52.95 82.075)
+		(start 42.2125 92)
+		(end 40.5 92)
 		(width 0.25)
 		(layer "F.Cu")
@@
 	)
 	(segment
-		(start 40.5 92)
-		(end 42.275 92)
+		(start 52.95 81.9375)
+		(end 52.95 82.075)
 		(width 0.25)
 		(layer "F.Cu")
@@
 		(polygon
 			(pts
-				(xy 38.65 81.6) (xy 38.65 82.25) (xy 42 82.3) (xy 42.65 83.15) (xy 42.65 87.705035) (xy 45.338585 93.739844)
-				(xy 51.3 93.75) (xy 51.3 96.4) (xy 52.4 96.4) (xy 52.4 94.2) (xy 54.6 94.2) (xy 54.6 92.35) (xy 46.175 92.35)
-				(xy 43.9 87.45) (xy 43.9 81.6)
+				(xy 38.65 81.6) (xy 38.65 82.25) (xy 42 82.3) (xy 42.65 83.15) (xy 42.65 87.518345) (xy 45.421821 93.739986)
+				(xy 51.3 93.75) (xy 51.3 96.4) (xy 52.4 96.4) (xy 52.4 94.2) (xy 54.6 94.2) (xy 54.6 92.35) (xy 46.26607 92.35)
+				(xy 43.9 87.253848) (xy 43.9 81.6)
 			)
 		)
