File: hardware/tag/_autosave-tag.kicad_sch (KiCad schematic)
At the start: 101 parts, among them J1 USB_C_Receptacle_USB2.0_16P, J2 BATTERY, J3 UART, J4 I2C, J5 STM SWD, J7 BLE SWD, J8 SOURCE, SW1 SW_Push, SW2 SW_SPDT, SW3 SW_Push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

Commit message: wip(hardware): save tag schematic & pcb layout
Parts:
- added TP5: TestPoint, TestPoint:TestPoint_Pad_D1.0mm, symbol Connector:TestPoint
- renumbered R24 to R22
Connections:
- net SPI_CS2: now also TP5.1
Other:
- moved on the sheet: R24, TP12, TP9
Changed lines of the file:
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@@
 	(wire
 		(pts
-			(xy 383.54 198.12) (xy 383.54 201.93)
+			(xy 383.54 219.71) (xy 383.54 223.52)
 		)
 		(stroke
@@
 	(wire
 		(pts
+			(xy 398.78 198.12) (xy 398.78 201.93)
+		)
+		(stroke
+			(width 0)
+			(type default)
+		)
+	)
+	(wire
+		(pts
 			(xy 171.45 165.1) (xy 171.45 166.37)
 		)
@@
 	(wire
 		(pts
-			(xy 398.78 198.12) (xy 398.78 201.93)
+			(xy 398.78 219.71) (xy 398.78 223.52)
 		)
 		(stroke
@@
 	)
 	(label "BLE_RX"
-		(at 398.78 198.12 90)
+		(at 398.78 219.71 90)
 		(effects
 			(font
@@
 		)
 	)
+	(label "SPI_CS2"
+		(at 398.78 198.12 90)
+		(effects
+			(font
+				(size 1.016 1.016)
+			)
+			(justify left bottom)
+		)
+	)
 	(label "PA10 {slash} UART1_RX"
 		(at 218.44 200.66 0)
@@
 	)
 	(label "BLE_TX"
-		(at 383.54 198.12 90)
+		(at 383.54 219.71 90)
 		(effects
 			(font
@@
 	(symbol
 		(lib_id "Connector:TestPoint")
-		(at 383.54 201.93 180)
+		(at 383.54 223.52 180)
 		(unit 1)
 		(exclude_from_sim no)
@@
 		(dnp no)
 		(property "Reference" "TP9"
-			(at 382.016 207.772 0)
+			(at 382.016 229.362 0)
 			(effects
 				(font
@@
 		)
 		(property "Value" "TestPoint"
-			(at 379.476 210.566 0)
+			(at 379.476 232.156 0)
 			(effects
 				(font
@@
 		)
 		(property "Footprint" "TestPoint:TestPoint_Pad_D1.0mm"
-			(at 378.46 201.93 0)
+			(at 378.46 223.52 0)
 			(effects
 				(font
@@
 		)
 		(property "Datasheet" "~"
-			(at 378.46 201.93 0)
+			(at 378.46 223.52 0)
 			(effects
 				(font
@@
 		)
 		(property "Description" "test point"
-			(at 383.54 201.93 0)
+			(at 383.54 223.52 0)
 			(effects
 				(font
@@
 	)
 	(symbol
+		(lib_id "Connector:TestPoint")
+		(at 398.78 201.93 180)
+		(unit 1)
+		(exclude_from_sim no)
+		(in_bom yes)
+		(on_board yes)
+		(dnp no)
+		(property "Reference" "TP5"
+			(at 397.002 207.772 0)
+			(effects
+				(font
+					(size 1.27 1.27)
+				)
+				(justify right)
+			)
+		)
+		(property "Value" "TestPoint"
+			(at 395.224 210.566 0)
+			(effects
+				(font
+					(size 1.27 1.27)
+				)
+				(justify right)
+			)
+		)
+		(property "Footprint" "TestPoint:TestPoint_Pad_D1.0mm"
+			(at 393.7 201.93 0)
+			(effects
+				(font
+					(size 1.27 1.27)
+				)
+				(hide yes)
+			)
+		)
+		(property "Datasheet" "~"
+			(at 393.7 201.93 0)
+			(effects
+				(font
+					(size 1.27 1.27)
+				)
+				(hide yes)
+			)
+		)
+		(property "Description" "test point"
+			(at 398.78 201.93 0)
+			(effects
+				(font
+					(size 1.27 1.27)
+				)
+				(hide yes)
+			)
+		)
+		(pin "1"
+		)
+		(instances
+			(project "tag"
+				(path "/36ff3ade-5474-48a6-a94c-a185611a6890"
+					(reference "TP5")
+					(unit 1)
+				)
+			)
+		)
+	)
+	(symbol
 		(lib_id "power:GND")
 		(at 30.48 271.78 0)
@@
 	(symbol
 		(lib_id "Device:R")
-		(at 379.73 68.58 0)
+		(at 307.34 160.02 0)
 		(unit 1)
 		(exclude_from_sim no)
@@
 		(on_board yes)
 		(dnp no)
-		(property "Reference" "R22"
-			(at 374.015 67.691 0)
+		(property "Reference" "R24"
+			(at 302.895 151.003 0)
 			(effects
 				(font
@@
 		)
 		(property "Value" "10k"
-			(at 377.698 69.85 0)
+			(at 306.578 153.162 0)
 			(effects
 				(font
@@
 		)
 		(property "Footprint" "Resistor_SMD:R_0603_1608Metric_Pad0.98x0.95mm_HandSolder"
-			(at 377.952 68.58 90)
+			(at 305.562 160.02 90)
 			(effects
 				(font
@@
 		)
 		(property "Datasheet" "~"
-			(at 379.73 68.58 0)
+			(at 307.34 160.02 0)
 			(effects
 				(font
@@
 		)
 		(property "Description" "Resistor"
-			(at 379.73 68.58 0)
+			(at 307.34 160.02 0)
 			(effects
 				(font
@@
 		)
 		(instances
-			(project "learningkcad"
+			(project "tag"
 				(path "/36ff3ade-5474-48a6-a94c-a185611a6890"
-					(reference "R22")
+					(reference "R24")
 					(unit 1)
 				)
@@
 	(symbol
 		(lib_id "Device:R")
-		(at 307.34 160.02 0)
+		(at 379.73 68.58 0)
 		(unit 1)
 		(exclude_from_sim no)
@@
 		(on_board yes)
 		(dnp no)
-		(property "Reference" "R24"
-			(at 302.895 151.003 0)
+		(property "Reference" "R22"
+			(at 374.015 67.691 0)
 			(effects
 				(font
@@
 		)
 		(property "Value" "10k"
-			(at 306.578 153.162 0)
+			(at 377.698 69.85 0)
 			(effects
 				(font
@@
 		)
 		(property "Footprint" "Resistor_SMD:R_0603_1608Metric_Pad0.98x0.95mm_HandSolder"
-			(at 305.562 160.02 90)
+			(at 377.952 68.58 90)
 			(effects
 				(font
@@
 		)
 		(property "Datasheet" "~"
-			(at 307.34 160.02 0)
+			(at 379.73 68.58 0)
 			(effects
 				(font
@@
 		)
 		(property "Description" "Resistor"
-			(at 307.34 160.02 0)
+			(at 379.73 68.58 0)
 			(effects
 				(font
@@
 		)
 		(instances
-			(project "tag"
+			(project "learningkcad"
 				(path "/36ff3ade-5474-48a6-a94c-a185611a6890"
-					(reference "R24")
+					(reference "R22")
 					(unit 1)
 				)
@@
 	(symbol
 		(lib_id "Connector:TestPoint")
-		(at 398.78 201.93 180)
+		(at 398.78 223.52 180)
 		(unit 1)
 		(exclude_from_sim no)
@@
 		(dnp no)
 		(property "Reference" "TP12"
-			(at 397.002 207.772 0)
+			(at 397.002 229.362 0)
 			(effects
 				(font
@@
 		)
 		(property "Value" "TestPoint"
-			(at 395.224 210.566 0)
+			(at 395.224 232.156 0)
 			(effects
 				(font
@@
 		)
 		(property "Footprint" "TestPoint:TestPoint_Pad_D1.0mm"
-			(at 393.7 201.93 0)
+			(at 393.7 223.52 0)
 			(effects
 				(font
@@
 		)
 		(property "Datasheet" "~"
-			(at 393.7 201.93 0)
+			(at 393.7 223.52 0)
 			(effects
 				(font
@@
 		)
 		(property "Description" "test point"
-			(at 398.78 201.93 0)
+			(at 398.78 223.52 0)
 			(effects
 				(font
