File: hardware/tag/_autosave-tag.kicad_sch (KiCad schematic)
At the start: 107 parts, among them J1 USB_C_Receptacle_USB2.0_16P, J2 BATTERY, J3 UART, J4 I2C, J5 STM SWD, J7 BLE SWD, J8 SOURCE, SW1 SW_Push, SW2 SW_SPDT, SW3 SW_Push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

Commit message: feat(hardware): Save tag schematic & pcb layout
Parts:
- added TP16: 3V3, TestPoint:TestPoint_Pad_D1.5mm, symbol Connector:TestPoint
- SW1: value SW_Push -> RESET
- SW2: value SW_SPDT -> BOOT
- SW3: value SW_Push -> USER
Connections:
- net +3.3V: now also TP16.1
Changed lines of the file:
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@@
 	(wire
 		(pts
+			(xy 398.78 219.71) (xy 398.78 223.52)
+		)
+		(stroke
+			(width 0)
+			(type default)
+		)
+	)
+	(wire
+		(pts
 			(xy 123.19 222.25) (xy 128.27 222.25)
 		)
@@
 	)
 	(symbol
+		(lib_id "Connector:TestPoint")
+		(at 398.78 223.52 180)
+		(unit 1)
+		(exclude_from_sim no)
+		(in_bom yes)
+		(on_board yes)
+		(dnp no)
+		(property "Reference" "TP16"
+			(at 397.002 229.362 0)
+			(effects
+				(font
+					(size 1.27 1.27)
+				)
+				(justify right)
+			)
+		)
+		(property "Value" "3V3"
+			(at 397.51 231.902 0)
+			(effects
+				(font
+					(size 1.27 1.27)
+				)
+				(justify right)
+			)
+		)
+		(property "Footprint" "TestPoint:TestPoint_Pad_D1.5mm"
+			(at 393.7 223.52 0)
+			(effects
+				(font
+					(size 1.27 1.27)
+				)
+				(hide yes)
+			)
+		)
+		(property "Datasheet" "~"
+			(at 393.7 223.52 0)
+			(effects
+				(font
+					(size 1.27 1.27)
+				)
+				(hide yes)
+			)
+		)
+		(property "Description" "test point"
+			(at 398.78 223.52 0)
+			(effects
+				(font
+					(size 1.27 1.27)
+				)
+				(hide yes)
+			)
+		)
+		(pin "1"
+		)
+		(instances
+			(project "tag"
+				(path "/36ff3ade-5474-48a6-a94c-a185611a6890"
+					(reference "TP16")
+					(unit 1)
+				)
+			)
+		)
+	)
+	(symbol
 		(lib_id "Device:FerriteBead")
 		(at 231.14 157.48 90)
@@
 			)
 		)
-		(property "Value" "SW_Push"
+		(property "Value" "RESET"
 			(at 124.968 182.88 90)
 			(effects
@@
 	)
 	(symbol
+		(lib_id "power:+3.3V")
+		(at 398.78 219.71 0)
+		(mirror y)
+		(unit 1)
+		(exclude_from_sim no)
+		(in_bom yes)
+		(on_board yes)
+		(dnp no)
+		(property "Reference" "#PWR058"
+			(at 398.78 223.52 0)
+			(effects
+				(font
+					(size 1.27 1.27)
+				)
+				(hide yes)
+			)
+		)
+		(property "Value" "+3.3V"
+			(at 398.78 215.646 0)
+			(effects
+				(font
+					(size 1.27 1.27)
+				)
+			)
+		)
+		(property "Footprint" ""
+			(at 398.78 219.71 0)
+			(effects
+				(font
+					(size 1.27 1.27)
+				)
+				(hide yes)
+			)
+		)
+		(property "Datasheet" ""
+			(at 398.78 219.71 0)
+			(effects
+				(font
+					(size 1.27 1.27)
+				)
+				(hide yes)
+			)
+		)
+		(property "Description" "Power symbol creates a global label with name \"+3.3V\""
+			(at 398.78 219.71 0)
+			(effects
+				(font
+					(size 1.27 1.27)
+				)
+				(hide yes)
+			)
+		)
+		(pin "1"
+		)
+		(instances
+			(project "tag"
+				(path "/36ff3ade-5474-48a6-a94c-a185611a6890"
+					(reference "#PWR058")
+					(unit 1)
+				)
+			)
+		)
+	)
+	(symbol
 		(lib_id "Connector:TestPoint")
 		(at 373.38 157.48 180)
@@
 	)
 	(symbol
-		(lib_id "Graphic:SYM_ESD_Large")
-		(at 185.42 123.19 0)
-		(unit 1)
-		(exclude_from_sim no)
-		(in_bom no)
-		(on_board no)
-		(dnp no)
-		(fields_autoplaced yes)
-		(property "Reference" "#SYM1"
-			(at 185.42 118.11 0)
-			(effects
-				(font
-					(size 1.27 1.27)
-				)
-				(hide yes)
-			)
-		)
-		(property "Value" "SYM_ESD_Large"
-			(at 185.42 129.54 0)
-			(effects
-				(font
-					(size 1.27 1.27)
-				)
-				(hide yes)
-			)
-		)
-		(property "Footprint" "Symbol:ESD-Logo_6.6x6mm_SilkScreen"
-			(at 185.293 123.952 0)
-			(effects
-				(font
-					(size 1.27 1.27)
-				)
-				(hide yes)
-			)
-		)
-		(property "Datasheet" "~"
-			(at 185.293 123.952 0)
-			(effects
-				(font
-					(size 1.27 1.27)
-				)
-				(hide yes)
-			)
-		)
-		(property "Description" "ESD warning/\"Do not touch\" symbol, large"
-			(at 185.42 123.19 0)
-			(effects
-				(font
-					(size 1.27 1.27)
-				)
-				(hide yes)
-			)
-		)
-		(property "Sim.Enable" "0"
-			(at 185.42 123.19 0)
-			(effects
-				(font
-					(size 1.27 1.27)
-				)
-				(hide yes)
-			)
-		)
-		(instances
-			(project ""
-				(path "/36ff3ade-5474-48a6-a94c-a185611a6890"
-					(reference "#SYM1")
-					(unit 1)
-				)
-			)
-		)
-	)
-	(symbol
 		(lib_id "power:GND")
 		(at 38.1 271.78 0)
@@
 			)
 		)
-		(property "Value" "SW_Push"
+		(property "Value" "USER"
 			(at 217.678 243.84 90)
 			(effects
@@
 			)
 		)
-		(property "Value" "SW_SPDT"
+		(property "Value" "BOOT"
 			(at 165.1 186.69 0)
 			(effects
