File: hardware/anchor/anchor.kicad_sch (KiCad schematic)
At the start: 94 parts, among them J2 USB_C_Receptacle_USB2.0_16P, J3 STM SWD, J4 BLE SWD, J5 BATTERY, SW1 SW_DIP_x03, SW2 RESET, SW3 BOOT, SW4 USER, U1 BQ24075RGT, U2 TPS63070RNMR, U3 USBLC6-2SC6, U4 STM32F411CEUx, U6 FSC-BT630, Y1 NX3225SA-24MHz

Commit message: update(hw): Apply design changes to anchor
Parts:
- removed C12: DNP, Capacitor_SMD:C_0805_2012Metric_Pad1.18x1.45mm_HandSolder, symbol Device:C
- removed C22: 100n, Capacitor_SMD:C_0603_1608Metric_Pad1.08x0.95mm_HandSolder, symbol Device:C
- removed C23, C3: 10u, Capacitor_SMD:C_0805_2012Metric_Pad1.18x1.45mm_HandSolder, symbol Device:C
- removed C6, C7: 4.7u, Capacitor_SMD:C_0805_2012Metric_Pad1.18x1.45mm_HandSolder, symbol Device:C
- removed D1: RED, LED_SMD:LED_0603_1608Metric_Pad1.05x0.95mm_HandSolder, symbol Device:LED
- removed J5: BATTERY, Other_Footprint:JST_BM02B-SRSS-TB_LF__SN_, symbol BM02B-SRSS-TB_LF__SN_:BM02B-SRSS-TB_LF__SN_
- removed R10: 6k, Resistor_SMD:R_0603_1608Metric_Pad0.98x0.95mm_HandSolder, symbol Device:R
- removed R9: 10k, Resistor_SMD:R_0603_1608Metric_Pad0.98x0.95mm_HandSolder, symbol Device:R
- removed SW3: BOOT, Button_Switch_SMD:SW_SPDT_PCM12, symbol Switch:SW_SPDT
- removed TP2: GND, TestPoint:TestPoint_Pad_D1.5mm, symbol Connector:TestPoint
- removed U6: FSC-BT630, Other_Footprint:FSC-BT630, symbol FSC-BT630_Generic_20P:FSC-BT630_Named_20P
- added C11, C15: 10u, Capacitor_SMD:C_0805_2012Metric_Pad1.18x1.45mm_HandSolder, symbol Device:C
- added C17, C5: 100n, Capacitor_SMD:C_0603_1608Metric_Pad1.08x0.95mm_HandSolder, symbol Device:C
- added C24, C26: DNP, Capacitor_SMD:C_01005_0402Metric, symbol Device:C_Small
- added C8: 1u, Capacitor_SMD:C_0603_1608Metric_Pad1.08x0.95mm_HandSolder, symbol Device:C
- added C9: 4.7u, Capacitor_SMD:C_0805_2012Metric_Pad1.18x1.45mm_HandSolder, symbol Device:C
- added D3: YELLOW, LED_SMD:LED_0603_1608Metric_Pad1.05x0.95mm_HandSolder, symbol Device:LED
- added J1: BATTERY, Other_Footprint:JST_BM02B-SRSS-TB_LF__SN_, symbol BM02B-SRSS-TB_LF__SN_:BM02B-SRSS-TB_LF__SN_
- added J3: BLE_Conn, Connector_Coaxial:U.FL_Hirose_U.FL-R-SMT-1_Vertical, symbol Connector:Conn_Coaxial_Small
- added L2: DNP, Inductor_SMD:L_0402_1005Metric, symbol Device:L
- added Q1: AO664, Package_SO:TSOP-6_1.65x3.05mm_P0.95mm, symbol Transistor_FET:IRF7309PBF
- added R12, R13, R7: 10k, Resistor_SMD:R_0603_1608Metric_Pad0.98x0.95mm_HandSolder, symbol Device:R
- added R19, R21: 2.2k, Resistor_SMD:R_0603_1608Metric_Pad0.98x0.95mm_HandSolder, symbol Device:R
- added SW1: PWR, Button_Switch_SMD:SW_Push_1P1T-MP_NO_Horizontal_Alps_SKRTLAE010, symbol Switch:SW_Push_Shielded
- added TP16: SYS, TestPoint:TestPoint_Pad_D1.5mm, symbol Connector:TestPoint
- added U1: MAX17048G_T10, Package_SON:SON-8-1EP_3x2mm_P0.5mm_EP1.4x1.6mm, symbol MAX17048G_T10:MAX17048G_T10
- added U5: FSC-BT630, other_footprint:FSC-BT630, symbol FSC-BT630:FSC-BT630_Named_20P
- D2: value YELLOW -> GREEN
- D4: renamed from D3; value YELLOW -> GREEN
- D5: renamed from D4; value GREEN -> RED
- R11: value 6k -> 100k
- renumbered C9 to C10, C10 to C12, C11 to C13, C13 to C16, C14 to C18, C15 to C19, C16 to C20, C17 to C21, C18 to C22, C19 to C23, C20 to C25, C21 to C27, C24 to C28, C25 to C29, C26 to C30, C8 to C6, C5 to C7, D7 to D1, D5 to D6, D6 to D7, J3 to J4, J4 to J5, R14 to R10, R15 to R14, R16 to R15, R17 to R16, R18 to R17, R19 to R18, R4 to R2, R21 to R22, R3 to R23, R22 to R24, R23 to R25, R24 to R26, R7 to R3, R2 to R4, R8 to R5, R5 to R6, R12 to R8, R13 to R9, SW1 to SW2, SW2 to SW3, TP9 to TP10, TP15 to TP11, TP10 to TP12, TP11 to TP13, TP12 to TP14, TP13 to TP7, TP7 to TP8, TP8 to TP9, U1 to U4, U4 to U6
Connections:
- net +3.3V: now also C15.1, C17.1, U5.7 (VDD)
- net +BATT: now also C5.1, C9.1, J1.1, U1.3 (VDD)
- net BLE_RST: now also U5.6 (RESET)
- net BLE_RX: now also U5.1 (UART_TX)
- net BLE_SWDCLK: now also U5.9 (SWDCLK)
- net BLE_SWDIO: now also U5.10 (SWDIO)
- net BLE_TX: now also U5.2 (UART_RX)
- net GND: now also D2.1 (K), R18.1, C11.2, C15.2, C17.2, C24.2, C26.2, C5.2, C8.1, C9.2, D3.1 (K), J1.2, J1.S1 (SHIELD), J1.S2 (SHIELD), J3.2 (Ext), Q1.5 (S1), R7.1, SW1.MP (B), U1.1 (CTG), U1.4 (GND), U1.6 (QSTRT), U1.9 (EP), U5.19 (GND1), U5.8 (GND0)
- net SYS: now also C11.1, Q1.2 (S2), R12.2, TP16.1
- net at D2.2 (A): now also R19.1
- net at U4.1 (TS): now also R7.2
- net LED_PM: now reaches U6.38 (PA15)
- net LED_PM: now also R21.2
- net PB9 / I2C1_SDA: now reaches U6.45 (PB8)
- net PB9 / I2C1_SDA: now also U1.8 (SDA)
- net PB8 / I2C1_SCL: now reaches U6.46 (PB9)
- net PB8 / I2C1_SCL: now also U1.7 (SCL)
- net at R11.1: now also C8.2, SW1.1
- net CHG: no longer names the net of U4.9 (~{CHG})
- net CHG: no longer D2.1 (K)
- net PGOOD: no longer names the net of R11.2
- net PGOOD: now also Q1.3 (G2), Q1.6 (S1), R12.1; no longer U4.7 (~{PGOOD})
- new net: D3.2 (A), R21.1
- new net: C24.1, L2.1, U5.20 (EXT_ANT)
- new net: Q1.1 (G1), R13.1, SW1.2
- new net: C26.1, J3.1 (In), L2.2
- new net: R19.2, U5.15 (P0.03)
- new net LOAD: Q1.4 (D2), R13.2
- no-connect marks 37 -> 36
Other:
- note added: "AO664"
- note added: "PI Filter"
- note added: "TRACE 50 Ohm !"
- moved on the sheet: C1, C10, C12, C13, C16, C18, C19, C2, C20, C21, C22, C23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

Commit message: feat: Release final hardware for tag & anchor
Parts:
- removed C8: 1u, Capacitor_SMD:C_0603_1608Metric_Pad1.08x0.95mm_HandSolder, symbol Device:C
- removed D3: YELLOW, LED_SMD:LED_0603_1608Metric_Pad1.05x0.95mm_HandSolder, symbol Device:LED
- removed J4: STM SWD, Other_Footprint:JST_BM04B-SRSS-TB_LF__SN_, symbol BM04B-SRSS-TB_LF__SN_:BM04B-SRSS-TB_LF__SN_
- removed Q1: AO664, Package_SO:TSOP-6_1.65x3.05mm_P0.95mm, symbol Transistor_FET:IRF7309PBF
- added C3: 100n, Capacitor_SMD:C_0603_1608Metric_Pad1.08x0.95mm_HandSolder, symbol Device:C
- added D4: GREEN, LED_SMD:LED_0603_1608Metric_Pad1.05x0.95mm_HandSolder, symbol Device:LED
- added J10: Conn_01x02, Connector_Wire:SolderWire-0.1sqmm_1x02_P3.6mm_D0.4mm_OD1mm, symbol Connector_Generic:Conn_01x02
- added J4: BM06B-SRSS-TB_LF__SN_, Connector_JST:JST_SH_BM06B-SRSS-TB_1x06-1MP_P1.00mm_Vertical, symbol BM06B-SRSS:BM06B-SRSS-TB_LF__SN_
- added J6: I2C, Other_Footprint:JST_BM04B-SRSS-TB_LF__SN_, symbol BM04B-SRSS-TB_LF__SN_:BM04B-SRSS-TB_LF__SN_
- added Q2: AO3404A, Package_TO_SOT_SMD:SOT-23, symbol Transistor_FET:AO3400A
- added Q3: AO3407A, Package_TO_SOT_SMD:SOT-23, symbol Transistor_FET:AO3401A
- added R27, R28: 10k, Resistor_SMD:R_0603_1608Metric_Pad0.98x0.95mm_HandSolder, symbol Device:R
- R11: value 100k -> 10k
- R12: value 10k -> 100k
- TP10: value TestPoint -> TX
- TP12: value TestPoint -> MISO
- TP13: value TestPoint -> CS1
- TP14: value TestPoint -> RX
- TP3: footprint TestPoint:TestPoint_Pad_D1.0mm -> TestPoint:TestPoint_Pad_D1.5mm
- TP4: footprint TestPoint:TestPoint_Pad_D1.5mm -> TestPoint:TestPoint_Pad_1.0x1.0mm
- TP8: value TestPoint -> SCK
- TP9: value TestPoint -> MOSI
- renumbered D4 to D3
Connections:
- net +3.3V: now also J5.5, J4.5, J6.1, R27.1, R28.1; no longer J5.1, R22.2
- net +BATT: now also J10.2 (Pin_2)
- net BLE_RST: now also J5.3; no longer J5.2
- net BLE_SWDCLK: now also J5.1; no longer J5.3
- net BLE_SWDIO: now also J5.2; no longer J5.4
- net GND: now also D3.1 (K), J5.4, C3.1, J10.1 (Pin_1), J4.6, J4.S1 (SHIELD), J4.S2 (SHIELD), J6.2, J6.S1 (SHIELD), J6.S2 (SHIELD), Q2.2 (S); no longer J5.5, U4.4 (~{CE})
- net LED_USR: now also R22.2; no longer D3.1 (K)
- net LOAD: now also C1.1, C2.1, C4.1, R1.2, R11.2, R2.2, U2.12_13 (VIN), Q3.3 (D); no longer R13.2
- net PB8 / I2C1_SCL: now also U6.45 (PB8), J6.3, R27.2; no longer U6.46 (PB9)
- net PB9 / I2C1_SDA: now also U6.46 (PB9), J6.4, R28.2; no longer U6.45 (PB8)
- net STM_SWDCLK: now also J4.3
- net STM_SWDIO: now also J4.4
- net SYS: now also R13.2, R21.2, Q3.2 (S); no longer C1.1, C2.1, C4.1, R1.2, R12.2, R2.2, U2.12_13 (VIN)
- net at SW1.1: now also R12.1, C3.2; no longer R11.1
- net at R21.1: now also D4.2 (A)
- net at R13.1: now also R12.2, Q2.3 (D), Q3.1 (G); no longer SW1.2
- net CHG: now reaches U4.9 (~{CHG})
- net CHG: now also D4.1 (K)
- net PA9 / UART1_TX: now reaches U6.30 (PA9)
- net PA9 / UART1_TX: now also J4.2
- net PA10 / UART1_RX: now reaches U6.31 (PA10)
- net PA10 / UART1_RX: now also J4.1
- net LED_PM renamed CHARGE_EN
- net CHARGE_EN: now also U4.4 (~{CE}); no longer R21.2
- new net: Q2.1 (G), R11.1, SW1.2
- no-connect marks 36 -> 33
Other:
- note removed: "AO664"
- moved on the sheet: H1, H2, H3, H4, J1, J5, TP1, TP10, TP11, TP12, TP13, TP14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

Commit message: feat: release final final hardware for tag + anchor
Parts:
- added D9: MBR230LSFT1G, Diode_SMD:D_SOD-123, symbol Device:D_Schottky
- added R29: 1k(TBD), Resistor_SMD:R_0603_1608Metric, symbol Device:R
- added R30: 10k, Resistor_SMD:R_0603_1608Metric, symbol Device:R
- C1, C10, C11, C12, C13, C2, C7, C9: footprint Capacitor_SMD:C_0805_2012Metric_Pad1.18x1.45mm_HandSolder -> Capacitor_SMD:C_0805_2012Metric
- C24, C26: footprint Capacitor_SMD:C_01005_0402Metric -> Capacitor_SMD:C_0402_1005Metric
- C3: value 100n -> 100n(TBD); footprint Capacitor_SMD:C_0603_1608Metric_Pad1.08x0.95mm_HandSolder -> Capacitor_SMD:C_0603_1608Metric
- C4, C5, C6: footprint Capacitor_SMD:C_0603_1608Metric_Pad1.08x0.95mm_HandSolder -> Capacitor_SMD:C_0603_1608Metric
- R1, R10, R11, R12, R13, R2, R21, R4, R6, R7: footprint Resistor_SMD:R_0603_1608Metric_Pad0.98x0.95mm_HandSolder -> Resistor_SMD:R_0603_1608Metric
Connections:
- net CHARGE_EN: now also R30.1
- net GND: now also R29.2, R30.2
- net LOAD: now also D9.1 (K); no longer Q3.3 (D), R11.2
- new net: D9.2 (A), Q3.3 (D), R11.2, R29.1

Commit message: Update: schematic with new dimensions and additional notes
Parts:
- D1: value ESD -> MBR230LSFT1G
Connections:
- net PWR_LATCH: now reaches Q2.1 (G), R11.1, SW1.2
- net PWR_LATCH: now also U6.39 (PB3)
- no-connect marks 33 -> 32
Other:
- note added: "NOTE: Use a 5 V-tolerant MCU GPIO. Configure the pin as open-drain."
- note added: "PWR_LATCH low = power off."
Changed lines of the file:
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@@
 	(rectangle
 		(start 21.59 78.74)
-		(end 165.1 179.07)
+		(end 176.53 179.07)
 		(stroke
 			(width 0)
@@
 		)
 	)
+	(text "NOTE: Use a 5 V-tolerant MCU GPIO.\n	  Configure the pin as open-drain.\n"
+		(exclude_from_sim no)
+		(at 151.384 105.156 0)
+		(effects
+			(font
+				(size 0.762 0.762)
+			)
+			(justify left)
+		)
+	)
 	(text "TRACE 50 Ohm !"
 		(exclude_from_sim no)
@@
 		)
 	)
+	(text "PWR_LATCH low = power off."
+		(exclude_from_sim no)
+		(at 155.448 107.696 0)
+		(effects
+			(font
+				(size 0.762 0.762)
+			)
+			(justify left)
+		)
+	)
 	(junction
 		(at 210.82 146.05)
@@
 	)
 	(no_connect
-		(at 237.49 201.93)
-	)
-	(no_connect
 		(at 237.49 186.69)
 	)
@@
 	(wire
 		(pts
-			(xy 228.6 207.01) (xy 237.49 207.01)
+			(xy 223.52 207.01) (xy 237.49 207.01)
 		)
 		(stroke
@@
 	(wire
 		(pts
-			(xy 228.6 184.15) (xy 237.49 184.15)
+			(xy 223.52 184.15) (xy 237.49 184.15)
 		)
 		(stroke
@@
 	(wire
 		(pts
+			(xy 223.52 201.93) (xy 237.49 201.93)
+		)
+		(stroke
+			(width 0)
+			(type default)
+		)
+	)
+	(wire
+		(pts
 			(xy 123.19 170.18) (xy 123.19 171.45)
 		)
@@
 	(wire
 		(pts
-			(xy 229.87 222.25) (xy 237.49 222.25)
+			(xy 223.52 222.25) (xy 237.49 222.25)
 		)
 		(stroke
@@
 	(wire
 		(pts
+			(xy 151.13 101.6) (xy 157.48 101.6)
+		)
+		(stroke
+			(width 0)
+			(type default)
+		)
+	)
+	(wire
+		(pts
 			(xy 74.93 224.79) (xy 74.93 231.14)
 		)
@@
 	(wire
 		(pts
-			(xy 228.6 212.09) (xy 237.49 212.09)
+			(xy 223.52 212.09) (xy 237.49 212.09)
 		)
 		(stroke
@@
 	(wire
 		(pts
-			(xy 228.6 199.39) (xy 237.49 199.39)
+			(xy 223.52 199.39) (xy 237.49 199.39)
 		)
 		(stroke
@@
 	(wire
 		(pts
-			(xy 228.6 209.55) (xy 237.49 209.55)
+			(xy 223.52 209.55) (xy 237.49 209.55)
 		)
 		(stroke
@@
 	)
 	(label "DIP3"
-		(at 228.6 212.09 0)
+		(at 223.52 212.09 0)
 		(effects
 			(font
@@
 	)
 	(label "UWB_RST"
-		(at 228.6 199.39 0)
+		(at 223.52 199.39 0)
 		(effects
 			(font
@@
 	)
 	(label "LED_USR"
-		(at 228.6 184.15 0)
+		(at 223.52 184.15 0)
 		(effects
 			(font
@@
 		)
 	)
+	(label "PWR_LATCH"
+		(at 157.48 101.6 0)
+		(effects
+			(font
+				(size 1 1)
+			)
+			(justify left bottom)
+		)
+	)
 	(label "PA0{slash}BTN_USR"
 		(at 297.18 226.06 180)
@@
 	)
 	(label "SPI_CS1"
-		(at 229.87 222.25 0)
+		(at 223.52 222.25 0)
 		(effects
 			(font
@@
 	)
 	(label "DIP1"
-		(at 228.6 207.01 0)
+		(at 223.52 207.01 0)
 		(effects
 			(font
@@
 	)
 	(label "DIP2"
-		(at 228.6 209.55 0)
+		(at 223.52 209.55 0)
 		(effects
 			(font
@@
 		)
 	)
+	(label "PWR_LATCH"
+		(at 223.52 201.93 0)
+		(effects
+			(font
+				(size 1 1)
+			)
+			(justify left bottom)
+		)
+	)
 	(label "USB_OTG_DM"
 		(at 285.75 194.31 180)
@@
 			)
 		)
-		(property "Value" "ESD"
+		(property "Value" "MBR230LSFT1G"
 			(at 93.98 214.6299 90)
 			(effects
